File: Eltraco Eagle/Single Turnout /Single Turnoutv0.2.brd (EAGLE design)
At the start: 100 x 80 mm, 80 parts, among them K1 NA, K2 NA, T1 BC547, T2 BC547, T3 BC547, T4 BC547

Commit message: New version PCB files and extra PCBs
Value of components printed on PCB. Current sensor, hall sensor and
relais add-on PCB added
Parts:
- removed U$10: (no value), holes:3,2
- added U$7: (no value), holes:3,2
- moved U$3 3.81 mm to (34.3, 29.2)
Changed lines of the file:
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@@
 </element>
 <element name="U$1" library="holes" package="3,2" value="" x="7.62" y="73.66" smashed="yes"/>
-<element name="U$3" library="holes" package="3,2" value="" x="34.29" y="33.02" smashed="yes"/>
 <element name="DC-DC" library="pinhead" package="1X04" value="" x="3.81" y="39.37" smashed="yes" rot="R270">
 <attribute name="NAME" x="5.6388" y="41.9862" size="1.27" layer="25" ratio="10" rot="R270"/>
@@
 <element name="U$4" library="holes" package="3,2" value="" x="58.42" y="73.66" smashed="yes"/>
 <element name="U$9" library="holes" package="3,2" value="" x="85.09" y="73.66" smashed="yes"/>
-<element name="U$10" library="holes" package="3,2" value="" x="85.09" y="33.02" smashed="yes"/>
 <element name="LO" library="pinhead" library_urn="urn:adsk.eagle:library:325" package="1X06" value="" x="10.16" y="13.97" smashed="yes">
 <attribute name="NAME" x="2.4638" y="15.7988" size="1.27" layer="25" ratio="10"/>
@@
 <element name="U$5" library="holes" package="3,2" value="" x="34.29" y="8.89" smashed="yes"/>
 <element name="U$6" library="holes" package="3,2" value="" x="85.09" y="8.89" smashed="yes"/>
+<element name="U$3" library="holes" package="3,2" value="" x="34.29" y="29.21" smashed="yes"/>
+<element name="U$7" library="holes" package="3,2" value="" x="85.09" y="29.21" smashed="yes"/>
 </elements>
 <signals>
